File: hardware/bridge.brd (EAGLE design)
At the start: 37.8 x 80 mm, 21 parts, among them IC1 MAX3232CPE, J1 RJ11, U1 MC34063ABN

Commit message: Minor design and documentation changes
Parts:
- removed U1: MC34063ABN, ST Microelctronics_By_element14_Batch_1:DIP254P762X480-8
- added IC2: MC34063AP, v-reg-3:DIL-08
- C3: value 0.1u -> 100u; device rcl:C025-024X044 -> rcl:E2,5-6E
- C7: value 100u -> 0.1u; device rcl:E2,5-6E -> rcl:C025-024X044
- D1: value 1N5819-B -> 1N4148; device diode:DO41-7.6 -> SparkFun-DiscreteSemi:DIODE-1N4148
- D2: value 1N4148DO35-7 -> 1N5819-B; device diode:DO35-7 -> diode:DO41-7.6
- R2: value 11k -> 1
- R4: value 1 -> 11k
- moved C3 25.4 mm to (35.6, 26.7), turned to 90 degrees
- moved D1 23.4 mm to (35.6, 19.1), turned to 90 degrees
- moved D2 23.4 mm to (12.7, 24.1)
- moved C7 23.4 mm to (17.8, 41.9), turned to 270 degrees
- moved R2 10.9 mm to (30.5, 26.7), turned to 270 degrees
- moved R4 10.9 mm to (21.6, 20.3), turned to 180 degrees
- moved C6 10.2 mm to (27.9, 41.9)
- moved C4 8.98 mm to (15.2, 41.9), turned to 270 degrees
- moved C5 4.02 mm to (24.1, 43.2), turned to 0 degrees
- moved R3 1.80 mm to (25.4, 19.1), turned to 270 degrees
- turned R1 to 270 degrees
Connections:
- removed net 12V: C7.+, D2.C, R1.1, R4.1, U1.6
- removed net N$1: R2.1, R3.1, U1.5
- new net N$16: IC2.1, IC2.7, IC2.8, R1.1, R2.1
- new net N$18: IC2.5, R3.1, R4.1
- net GND: now also C3.-, C7.2, D2.A, IC2.4, R4.2; no longer C5.2, C7.-, D1.A, R2.2, U1.4
- net N$10: now also C5.1; no longer C4.1
- net N$11: now also C5.2; no longer C4.2
- net N$12: now also C6.1; no longer C5.1
- net N$13: now also C7.1; no longer C6.1
- net N$17: now also D1.A; no longer D2.A
- net N$2: now also C3.+, D1.C, IC2.6, R2.2; no longer R4.2, U1.1, U1.7, U1.8
- net N$3: now also IC2.3; no longer U1.3
- net N$5: now also D2.C, IC2.2; no longer D1.C, U1.2
- net N$8: now also C4.2; no longer C3.2
- net N$9: now also C4.1; no longer C3.1
Routing:
- net N$16: track 0.00 -> 15.2 mm
- net 12V: track 12.7 -> 0.00 mm
- net N$18: track 0.00 -> 5.08 mm
- net N$1: track 5.08 -> 0.00 mm, vias 0 -> 1
- net N$8: track 2.54 -> 5.08 mm, vias 0 -> 1
- net N$2: track 15.2 -> 12.7 mm
- net GND: vias 0 -> 2
- net N$7: vias 0 -> 2
- net N$6: vias 0 -> 2
- net N$17: vias 0 -> 2

Commit message: Minor board beauty treatment
Parts:
- removed U$1: ESP01, esp8266modules:ESP01
- removed U$2: RJ9PTH, SparkFun-Connectors:RJ9
- added J2: RJ9PTH, SparkFun-Connectors:RJ9
- added M1: ESP01, esp8266modules:ESP01
- IC1: value MAX3232CPE -> MC34063AP; device maxim:DIL16 -> v-reg-3:DIL-08
- IC2: value MC34063AP -> MAX3232CPE; device v-reg-3:DIL-08 -> maxim:DIL16
- moved IC2 28.1 mm to (19.1, 54.6), turned to 0 degrees
- moved IC1 19.3 mm to (16.5, 31.8), turned to 270 degrees
- moved C6 7.18 mm to (22.9, 47.0)
- moved C7 7.18 mm to (12.7, 47.0)
- moved C4 7.18 mm to (10.2, 47.0)
- moved C1 7.18 mm to (10.2, 29.2)
- moved J1 7.18 mm to (25.4, 7.62)
- moved D2 7.18 mm to (7.62, 29.2)
- moved C3 7.18 mm to (30.5, 31.8)
- moved D1 7.18 mm to (30.5, 24.1)
- moved LED1 7.18 mm to (22.9, 41.9)
- moved R1 7.18 mm to (22.9, 31.8)
- moved R2 7.18 mm to (25.4, 31.8)
- moved C2 7.18 mm to (16.5, 40.6)
- moved C5 7.18 mm to (19.1, 48.3)
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Connections:
- net N$17 renamed VBATT
- removed net N$2: C3.+, D1.C, IC2.6, R1.2, R2.2
- removed net VCC: C2.+, IC1.16, L1.2, R3.2, R5.1, U$1.CH_PD, U$1.VCC
- new net 12V: C3.+, D1.C, IC1.6, R1.2, R2.2
- new net 3V3: C2.+, IC2.16, L1.2, M1.CH_PD, M1.VCC, R3.2, R5.1
- net GND: now also IC1.4, IC2.15, J2.1, J2.2, M1.GND; no longer IC1.15, IC2.4, U$1.GND, U$2.1, U$2.2
- net N$10: now also IC2.4; no longer IC1.4
- net N$11: now also IC2.5; no longer IC1.5
- net N$12: now also IC2.6; no longer IC1.6
- net N$13: now also IC2.2; no longer IC1.2
- net N$14: now also IC2.14, J2.3; no longer IC1.14, U$2.3
- net N$15: now also IC2.13, J2.4; no longer IC1.13, U$2.4
- net N$16: now also IC1.1, IC1.7, IC1.8; no longer IC2.1, IC2.7, IC2.8
- net N$18: now also IC1.5; no longer IC2.5
- net N$3: now also IC1.3; no longer IC2.3
- net N$5: now also IC1.2; no longer IC2.2
- net N$6: now also IC2.11, M1.TX; no longer IC1.11, U$1.TX
- net N$7: now also IC2.12, M1.RX; no longer IC1.12, U$1.RX
- net N$8: now also IC2.3; no longer IC1.3
- net N$9: now also IC2.1; no longer IC1.1
Routing:
- net 3V3: track 0.00 -> 56.1 mm
- net VCC: track 56.1 -> 0.00 mm
- net N$2: track 12.7 -> 0.00 mm
- net 12V: track 0.00 -> 12.7 mm
- net GND: track 153.5 -> 150.9 mm
- net N$6: track 4.53 -> 5.79 mm
Other:
- board size 37.8 x 80 mm -> 37.8 x 90.2 mm

Commit message: Small board changes
Parts:
- moved M1 79.0 mm to (74.9, 19.1), turned to 270 degrees
- moved IC2 50.3 mm to (54.6, 19.1), turned to 270 degrees
- moved C4 41.5 mm to (47.0, 27.9), turned to 180 degrees
- moved C5 41.3 mm to (48.3, 19.1), turned to 270 degrees
- moved C7 40.5 mm to (47.0, 25.4), turned to 180 degrees
- moved C6 39.9 mm to (47.0, 15.2), turned to 180 degrees
- moved LED1 32.8 mm to (41.9, 15.2), turned to 0 degrees
- moved L1 31.4 mm to (38.1, 30.5), turned to 0 degrees
- moved C2 31.0 mm to (41.9, 22.9)
- moved R5 26.9 mm to (38.1, 19.1), turned to 270 degrees
- moved J1 25.1 mm to (7.62, 25.4), turned to 270 degrees
- moved C3 24.2 mm to (31.8, 7.62), turned to 0 degrees
- moved D2 21.6 mm to (29.2, 30.5), turned to 180 degrees
- moved R2 20.1 mm to (31.8, 12.7), turned to 180 degrees
- moved C1 19.1 mm to (29.2, 27.9), turned to 180 degrees
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Routing:
- net VBATT: track 8.41 -> 31.6 mm, vias 2 -> 0
- net GND: track 150.9 -> 136.7 mm, vias 2 -> 0
Other:
- board size 37.8 x 90.2 mm -> 88.9 x 38.1 mm
