File: hardware/bridge.sch (EAGLE design)
At the start: 21 parts, among them IC1 MAX3232CPE, J1 RJ11, U1 MC34063ABN

Commit message: Minor design and documentation changes
Parts:
- removed U1: MC34063ABN, ST Microelctronics_By_element14_Batch_1:MC34063ABN
- added IC2: MC34063AP, v-reg-3:MC34063AP
- C3: value 0.1u -> 100u; device rcl:C-US025-024X044 -> rcl:CPOL-USE2,5-6E
- C7: value 100u -> 0.1u; device rcl:CPOL-USE2,5-6E -> rcl:C-US025-024X044
- D1: value 1N5819-B -> 1N4148; device diode:1N5819-B -> SparkFun-DiscreteSemi:DIODE1N4148
- D2: value 1N4148DO35-7 -> 1N5819-B; device diode:1N4148DO35-7 -> diode:1N5819-B
- R2: value 11k -> 1
- R4: value 1 -> 11k
Connections:
- removed net 12V: C7.+, D2.C, R1.1, R4.1, U1.VCC
- removed net N$1: R2.1, R3.1, U1.CII
- new net N$16: IC2.DRC, IC2.IPK, IC2.SWC, R1.1, R2.1
- new net N$18: IC2.COMP, R3.1, R4.1
- net GND: now also C3.-, C7.2, D2.A, IC2.GND, R4.2; no longer C5.2, C7.-, D1.A, R2.2, U1.GND
- net N$10: now also C5.1; no longer C4.1
- net N$11: now also C5.2; no longer C4.2
- net N$12: now also C6.1; no longer C5.1
- net N$13: now also C7.1; no longer C6.1
- net N$17: now also D1.A; no longer D2.A
- net N$2: now also C3.+, D1.C, IC2.VCC, R2.2; no longer R4.2, U1.DRC, U1.IPK, U1.SWC
- net N$3: now also IC2.TC; no longer U1.TC
- net N$5: now also D2.C, IC2.SWE; no longer D1.C, U1.SWE
- net N$8: now also C4.2; no longer C3.2
- net N$9: now also C4.1; no longer C3.1
Other:
- moved on the sheet: C1, C2, C4, C5, C6, J1, R1, R2, R3, R4, U$2

Commit message: Minor board beauty treatment
Parts:
- IC1: value MAX3232CPE -> MC34063AP; device maxim:MAX3232CPE -> v-reg-3:MC34063AP
- IC2: value MC34063AP -> MAX3232CPE; device v-reg-3:MC34063AP -> maxim:MAX3232CPE
- renumbered U$1 to M1, U$2 to J2
Connections:
- net N$17 renamed VBATT
- removed net N$2: C3.+, D1.C, IC2.VCC, R1.2, R2.2
- removed net VCC: C2.+, IC1P.VCC, L1.2, M1.CH_PD, M1.VCC, R3.2, R5.1
- new net 12V: C3.+, D1.C, IC1.VCC, R1.2, R2.2
- new net 3V3: C2.+, IC2P.VCC, L1.2, M1.CH_PD, M1.VCC, R3.2, R5.1
- net GND: now also IC1.GND, IC2P.GND; no longer IC1P.GND, IC2.GND
- net N$10: now also IC2G$1.C2+; no longer IC1G$1.C2+
- net N$11: now also IC2G$1.C2-; no longer IC1G$1.C2-
- net N$12: now also IC2G$1.V-; no longer IC1G$1.V-
- net N$13: now also IC2G$1.V+; no longer IC1G$1.V+
- net N$14: now also IC2G$1.T1OUT; no longer IC1G$1.T1OUT
- net N$15: now also IC2G$1.R1IN; no longer IC1G$1.R1IN
- net N$16: now also IC1.DRC, IC1.IPK, IC1.SWC; no longer IC2.DRC, IC2.IPK, IC2.SWC
- net N$18: now also IC1.COMP; no longer IC2.COMP
- net N$3: now also IC1.TC; no longer IC2.TC
- net N$5: now also IC1.SWE; no longer IC2.SWE
- net N$6: now also IC2G$1.T1IN; no longer IC1G$1.T1IN
- net N$7: now also IC2G$1.R1OUT; no longer IC1G$1.R1OUT
- net N$8: now also IC2G$1.C1-; no longer IC1G$1.C1-
- net N$9: now also IC2G$1.C1+; no longer IC1G$1.C1+
